File: modules/EXPERIMENTAL-KICAD-10/02-vco/electronics/core/sheets/raw-oscillator.kicad_sch (KiCad schematic)
At the start: 56 parts, among them Q1 BC847BS, Q2 MMBT3906, Q3 J111, Q4 MMBFJ111, Q5 MMBT5551, U1 TL072, U2 TL072, U3 LM311

Commit message: Revert "Updated experimental VCO Core"
This reverts commit 34f3e113d18d89390407e9554ee904153359fd81.
Parts:
- Q1: footprint Package_TO_SOT_SMD:SOT-363_SC-70-6 -> Shmoergh_Custom_Footprints:SOT-363_SC-70-6
Changed lines of the file:
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@@
 			)
 		)
-		(property "Footprint" "Package_TO_SOT_SMD:SOT-363_SC-70-6"
+		(property "Footprint" "Shmoergh_Custom_Footprints:SOT-363_SC-70-6"
 			(at 172.72 72.39 0)
 			(hide yes)
@@
 			)
 		)
-		(property "Footprint" "Package_TO_SOT_SMD:SOT-363_SC-70-6"
+		(property "Footprint" "Shmoergh_Custom_Footprints:SOT-363_SC-70-6"
 			(at 172.72 72.39 0)
 			(hide yes)

Commit message: Updated experimental VCO Core
Parts:
- Q1: footprint Shmoergh_Custom_Footprints:SOT-363_SC-70-6 -> Package_TO_SOT_SMD:SOT-363_SC-70-6
Changed lines of the file:
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@@
 			)
 		)
-		(property "Footprint" "Shmoergh_Custom_Footprints:SOT-363_SC-70-6"
+		(property "Footprint" "Package_TO_SOT_SMD:SOT-363_SC-70-6"
 			(at 172.72 72.39 0)
 			(hide yes)
@@
 			)
 		)
-		(property "Footprint" "Shmoergh_Custom_Footprints:SOT-363_SC-70-6"
+		(property "Footprint" "Package_TO_SOT_SMD:SOT-363_SC-70-6"
 			(at 172.72 72.39 0)
 			(hide yes)
