File: modules/02-vco/electronics/KICAD-10-EXPERIMENTAL/core/sheets/power.kicad_sch (KiCad schematic)
At the start: 15 parts, among them J3 Conn_02x05_Odd_Even, J4 Conn_01x02, J5 Conn_02x03_Odd_Even, U7 TL072

Commit message: Reverted VCO Core back to latest stable
- The latest working version of the VCO is this: (commit: https://github.com/shmoergh/moduleur/tree/b8f2f3887ee0ce40083da4d1238f04f5c6e473fa). Somewhere
between January 24 and May 24 the PCB got corrupted and it doesn't work properly. It could be the KiCAD 10 migration.
Other:
- company: (none) -> Shmøergh
- title: (none) -> Moduleur VCO core
