File: modules/02-vco/electronics/KICAD-10-EXPERIMENTAL/core/sheets/waveshapers.kicad_sch (KiCad schematic)
At the start: 44 parts, among them U4 TL072, U5 TL072, U6 TL072

Commit message: Reverted VCO Core back to latest stable
- The latest working version of the VCO is this: (commit: https://github.com/shmoergh/moduleur/tree/b8f2f3887ee0ce40083da4d1238f04f5c6e473fa). Somewhere
between January 24 and May 24 the PCB got corrupted and it doesn't work properly. It could be the KiCAD 10 migration.
Other:
- company: (none) -> Shmøergh
- title: (none) -> Moduleur VCO core
