File: modules/02-vco/electronics/KiCAD9-BACKUP/core/sheets/power.kicad_sch (KiCad schematic)
At the start: 15 parts, among them J3 Conn_02x05_Odd_Even, J4 Conn_01x02, J5 Conn_02x03_Odd_Even, U7 TL072

Commit message: Fix: Replace generic MMBT3906 with ON Semi for Q2
Q2 is the actuator in the master current servo loop (U1B → Q2) that sets the tail current for the exponential converter. The previous BOM specified the generic LCSC part C7420354, which JLCPCB silently substituted between production batches: batch 1 (Jan 2026) received a working part, while batches 2 and 3 received Zhuhai Hongjiacheng (R+O) MMBT3906 parts under the same C-code.

The R+O datasheet only characterizes hFE at IC = −10 mA and above, with no minimum specified at low collector currents. The circuit operates Q2 at sub-milliamp currents, where the substituted part has insufficient gain to close the servo loop. U1B saturates against the negative supply rail trying to compensate, leaving Q2's collector current stuck at a fixed (too-low) value regardless of CV input.
Symptoms across all affected boards (20+ units, fully uniform):

- VCO pitch ceiling at ~70 Hz
- Pitch plateaus and flattens above a certain CV — no further response to increasing CV
- R_BIAS1 trim has no effect on output (loop railed)
- TP1 floats at ~1V instead of being servoed to 0V
- U1B output pinned at −10.3V (TL072 negative rail)

Verified by swapping Q2 with a verified-genuine 2N3906 on two broken boards — both immediately tracked V/oct correctly across full CV range.
The replacement part ON Semi MMBT3906LT1G (LCSC C53444) explicitly specifies hFE ≥ 60 at IC = −0.1 mA in its datasheet, guaranteeing correct behavior in this circuit's operating range.
Changes:

BOM: Q2 LCSC part number changed from C7420354 → C53444
Schematic annotation updated to specify ON Semi MMBT3906LT1G
Production note added: "Q2 (C53444): Do not substitute. Must be ON Semi MMBT3906LT1G."
Other:
- company: Shmøergh -> (none)
- title: Moduleur VCO core -> (none)
